Commit message: Add Oak 4-D visualization

File: python/foxglove-sdk-examples/rebotarm-demo/urdf/reBot-DevArm_description_fixend/urdf/reBot-DevArm_fixend.urdf (robot description, URDF)
Before this commit: robot reBot-DevArm_fixend, 8 links, 7 joints
Links:
- added link oak
- added link oak_model_origin; visual mesh filename=../meshes/OAK4-D.stl
Joints:
- added joint oak_model_origin_joint: type fixed, parent oak, child oak_model_origin, origin xyz=0 0 0 rpy=1.5708 0 1.5708
- added joint oak_mount_joint: type fixed, parent link5, child oak, origin xyz=0.0 0.0 0.06 rpy=0 0 0

Commit message: Properly orient Oak camera

File: python/foxglove-sdk-examples/rebotarm-demo/urdf/reBot-DevArm_description_fixend/urdf/reBot-DevArm_fixend.urdf (robot description, URDF)
Before this commit: robot reBot-DevArm_fixend, 10 links, 9 joints
Joints:
- joint oak_mount_joint: origin xyz=0.0 0.0 0.06 rpy=0 0 0 -> xyz=0.0320 0.0 -0.074 rpy=3.14159 0 0

Commit message: Add streaming of oak rgbd

File: python/foxglove-sdk-examples/rebotarm-demo/urdf/reBot-DevArm_description_fixend/urdf/reBot-DevArm_fixend.urdf (robot description, URDF)
Before this commit: robot reBot-DevArm_fixend, 10 links, 9 joints
Joints:
- joint oak_mount_joint: origin xyz=0.0320 0.0 -0.074 rpy=3.14159 0 0 -> xyz=0.0320 0.0 -0.08291 rpy=3.14159 0 0
